Commit message: finished base platform in urdf

File: mesh_bot_description/urdf/mesh_bot.urdf.xacro (robot description, xacro)
@@ -4,16 +4,22 @@
     xmlns:controller="http://playerstage.sourceforge.net/gazebo/xmlschema/#controller"
     xmlns:interface="http://playerstage.sourceforge.net/gazebo/xmlschema/#interface" >
-    <!-- all values are in inches and are converted to meters bellow -->
+    <!-- all values are in inches -->
     <property name="pi" value="3.1415"/>
     <property name="in_m" value="0.0254"/>
-    <property name="base_width" value="28"/>
-    <property name="base_length" value="40"/>
-    <property name="base_height" value="24"/>
-    <property name="base_clearance" value="9.5"/>
-    <property name="wheel_radius" value="8"/>
-    <property name="wheel_width" value="5"/>
-    <property name="wheel_setback" value="10"/>
-    <property name="wheel_block_height" value="1.5"/>
-    <property name="wheel_separation" value="21"/>
+    <property name="cos_2_3_pi" value="-0.5"/>
+    <property name="sin_2_3_pi" value="0.866025"/>
+    <property name="cos_4_3_pi" value="-0.5"/>
+    <property name="sin_4_3_pi" value="-0.866025"/>
+    <property name="base_radius" value="12"/>
+    <property name="base_height" value=".5"/>
+    <!-- motors are in inches -->
+    <property name="motor_height" value="2"/>
+    <property name="motor_width" value="2"/>
+    <property name="motor_length" value="4"/>
+    <property name="motor_placement_radius" value="6"/>
+    <!-- wheels are in inches-->
+    <property name="wheel_radius" value="2"/>
+    <property name="wheel_width" value="1"/>
+    <property name="wheel_axil_offset" value="1.5"/>
     <property name="castor_bar_height" value="6"/>
     <property name="castor_bar_width" value="4"/>
@@ -63,14 +69,14 @@
         </inertial>
         <visual>
-            <origin xyz="${-(base_length/2-wheel_setback)*in_m} 0 0" rpy="0 0 0" />
-            <geometry>
-                <box size="${base_length*in_m} ${base_width*in_m} 0.001" />
+            <origin xyz="0 0 0" rpy="0 0 0" />
+            <geometry>
+                <cylinder radius="${base_radius*in_m}" length = ".001"/>
             </geometry>
             <material name="Shadow" />
         </visual>
         <collision>
-            <origin xyz="${-(base_length/2-wheel_setback)*in_m} 0 0" rpy="0 0 0" />
-            <geometry>
-                <box size="${base_length*in_m} ${base_width*in_m} 0.001" />
+            <origin xyz="0 0 0" rpy="0 0 0" />
+            <geometry>
+                <cylinder radius="${base_radius*in_m}" length = ".01"/>
             </geometry>
         </collision>
@@ -79,83 +85,196 @@
     <link name="base_link">
         <inertial>
-            <mass value="50" />
-            <origin xyz="0 0 0.0" />
-            <inertia ixx="0.01" ixy="0.0" ixz="0.0"
-            iyy="0.01" iyz="0.0" izz="0.5" />
-        </inertial>
-        <visual>
-            <origin xyz="${-(base_length/2-wheel_setback)*in_m} 0 ${base_height/2*in_m}" rpy="0 0 0" />
-            <geometry>
-                <box size="${base_length*in_m} ${base_width*in_m} ${base_height*in_m}" />
-            </geometry>
-            <material name="Green" />
-        </visual>
-        <collision>
-            <origin xyz="${-(base_length/2-wheel_setback)*in_m} 0 ${base_height/2*in_m}" rpy="0 0 0" />
-            <geometry>
-                <box size="${base_length*in_m} ${base_width*in_m} ${base_height*in_m}" />
+          <mass value="5" />
+          <origin xyz="0 0 0" />
+          <inertia ixx="0.0001" ixy="0.0" ixz="0.0"
+                  iyy="0.0001" iyz="0.0"
+                  izz="0.0001" />
+        </inertial>
+        <visual>
+            <origin xyz="0 0 ${(base_height/2)*in_m}" rpy="0 0 0" />
+            <geometry>
+                <cylinder radius="${base_radius*in_m}" length = "${base_height*in_m}"/>
+            </geometry>
+            <material name="Grey" />
+        </visual>
+        <collision>
+            <origin xyz="0 0 ${(base_height/2)*in_m}" rpy="0 0 0" />
+            <geometry>
+                <cylinder radius="${base_radius*in_m}" length = "${base_height*in_m}"/>
             </geometry>
         </collision>
     </link>
     <joint name="base_footprint_joint" type="fixed">
-        <origin xyz="0 0 ${base_clearance*in_m}" rpy="0 0 0" />
+        <origin xyz="0 0 ${(motor_height/2 + wheel_radius)*in_m}" rpy="0 0 0" />
         <parent link="base_footprint"/>
         <child link="base_link" />
     </joint>
-    <!-- left wheel -->
-    <link name="left_wheel_link">
+    <!-- motor 0 -->
+    <link name="motor_0_link">
+        <inertial>
+          <mass value="2" />
+          <origin xyz="0 0 0" />
+          <inertia ixx="0.0001" ixy="0.0" ixz="0.0"
+                  iyy="0.0001" iyz="0.0"
+                  izz="0.0001" />
+        </inertial>
+        <visual>
+            <origin xyz="${-motor_length/2 * in_m} 0 0" rpy="0 0 0" />
+            <geometry>
+                <box size="${motor_length *in_m} ${motor_width*in_m} ${motor_height*in_m}" />
+            </geometry>
+            <material name="Black" />
+        </visual>
+        <collision>
+            <origin xyz="${-motor_length/2 * in_m} 0 0" rpy="0 0 0" />
+            <geometry>
+                <box size="${motor_length *in_m} ${motor_width*in_m} ${motor_height*in_m}" />
+            </geometry>
+        </collision>
+    </link>
+    <joint name="motor_0_joint" type="fixed">
+        <origin xyz="${motor_placement_radius * in_m} 0 ${-motor_height/2 *in_m}" rpy="0 0 0" />
+        <parent link="base_link"/>
+        <child link="motor_0_link" />
+    </joint>
+    <!-- wheel 0 -->
+    <link name="wheel_0_link">
         <inertial>
             <origin xyz="0 0 0"/>
-            <mass value="2" />
+            <mass value=".5" />
             <inertia ixx="0.001" ixy="0.0" ixz="0.0"
             iyy="0.001" iyz="0.0" izz="0.001" />
         </inertial>
         <visual>
-            <origin xyz="0 0 0" rpy="0 ${pi/2} ${pi/2}" />
-            <geometry>
-                <cylinder radius="${wheel_radius*in_m}" length = "${wheel_width*in_m}"/>
+            <origin xyz="0 0 0" rpy="0 ${pi/2} 0" />
+            <geometry>
+                <cylinder radius="${wheel_radius*in_m}" length = "${wheel_width*in_m}"/>
+            </geometry>
+            <material name="Green" />
+        </visual>
+        <collision>
+            <origin xyz="0 0 0" rpy="0 ${pi/2} 0" />
+            <geometry>
+                <cylinder radius="${wheel_radius*in_m}" length = "${wheel_width*in_m}"/>
+            </geometry>
+        </collision>
+    </link>
+    <joint name="wheel_0_joint" type="continuous">
+        <origin xyz="${wheel_axil_offset * in_m} 0 0" rpy="0 0 0"/>
+        <parent link="motor_0_link"/>
+        <child link="wheel_0_link"/>
+        <axis xyz="1 0 0"/>
+    </joint>
+    <!-- motor 1 -->
+    <link name="motor_1_link">
+        <inertial>
+          <mass value="2" />
+          <origin xyz="0 0 0" />
+          <inertia ixx="0.0001" ixy="0.0" ixz="0.0"
+                  iyy="0.0001" iyz="0.0"
+                  izz="0.0001" />
+        </inertial>
+        <visual>
+            <origin xyz="${-motor_length/2 * in_m} 0 0" rpy="0 0 0" />
+            <geometry>
+                <box size="${motor_length *in_m} ${motor_width*in_m} ${motor_height*in_m}" />
             </geometry>
             <material name="Black" />
         </visual>
         <collision>
-            <origin xyz="0 0 0" rpy="0 ${pi/2} ${pi/2}" />
-            <geometry>
-                <cylinder radius="${wheel_radius*in_m}" length = "${wheel_width*in_m}"/>
-            </geometry>
-        </collision>
-    </link>
-    <joint name="left_wheel_joint" type="continuous">
-        <origin xyz="0 ${-wheel_separation/2*in_m} ${-wheel_block_height*in_m} " rpy="0 0 0"/>
+            <origin xyz="${-motor_length/2 * in_m} 0 0" rpy="0 0 0" />
+            <geometry>
+                <box size="${motor_length *in_m} ${motor_width*in_m} ${motor_height*in_m}" />
+            </geometry>
+        </collision>
+    </link>
+    <joint name="motor_1_joint" type="fixed">
+        <origin xyz="${motor_placement_radius * cos_2_3_pi * in_m} ${motor_placement_radius * sin_2_3_pi *in_m} ${-motor_height/2 *in_m}" rpy="0 0 ${(2*pi)/3}" />
         <parent link="base_link"/>
-        <child link="left_wheel_link"/>
-        <axis xyz="0 1 0"/>
-    </joint>
-    <!-- right wheel -->
-    <link name="right_wheel_link">
+        <child link="motor_1_link" />
+    </joint>
+    <!-- wheel 1 -->
+    <link name="wheel_1_link">
         <inertial>
             <origin xyz="0 0 0"/>
-            <mass value="2" />
+            <mass value=".5" />
             <inertia ixx="0.001" ixy="0.0" ixz="0.0"
             iyy="0.001" iyz="0.0" izz="0.001" />
         </inertial>
         <visual>
-            <origin xyz="0 0 0" rpy="0 ${pi/2} ${pi/2}" />
-            <geometry>
-                <cylinder radius="${wheel_radius*in_m}" length = "${wheel_width*in_m}"/>
+            <origin xyz="0 0 0" rpy="0 ${pi/2} 0" />
+            <geometry>
+                <cylinder radius="${wheel_radius*in_m}" length = "${wheel_width*in_m}"/>
+            </geometry>
+            <material name="Green" />
+        </visual>
+        <collision>
+            <origin xyz="0 0 0" rpy="0 ${pi/2} 0" />
+            <geometry>
+                <cylinder radius="${wheel_radius*in_m}" length = "${wheel_width*in_m}"/>
+            </geometry>
+        </collision>
+    </link>
+    <joint name="wheel_1_joint" type="continuous">
+        <origin xyz="${wheel_axil_offset * in_m} 0 0" rpy="0 0 0"/>
+        <parent link="motor_1_link"/>
+        <child link="wheel_1_link"/>
+        <axis xyz="1 0 0"/>
+    </joint>
+    <!-- motor 2 -->
+    <link name="motor_2_link">
+        <inertial>
+          <mass value="2" />
+          <origin xyz="0 0 0" />
+          <inertia ixx="0.0001" ixy="0.0" ixz="0.0"
+                  iyy="0.0001" iyz="0.0"
+                  izz="0.0001" />
+        </inertial>
+        <visual>
+            <origin xyz="${-motor_length/2 * in_m} 0 0" rpy="0 0 0" />
+            <geometry>
+                <box size="${motor_length *in_m} ${motor_width*in_m} ${motor_height*in_m}" />
             </geometry>
             <material name="Black" />
         </visual>
         <collision>
-            <origin xyz="0 0 0" rpy="0 ${pi/2} ${pi/2}" />
-            <geometry>
-                <cylinder radius="${wheel_radius*in_m}" length = "${wheel_width*in_m}"/>
-            </geometry>
-        </collision>
-    </link>
-    <joint name="right_wheel_joint" type="continuous">
-        <origin xyz="0 ${wheel_separation/2*in_m} ${-wheel_block_height*in_m} " rpy="0 0 0"/>
+            <origin xyz="${-motor_length/2 * in_m} 0 0" rpy="0 0 0" />
+            <geometry>
+                <box size="${motor_length *in_m} ${motor_width*in_m} ${motor_height*in_m}" />
+            </geometry>
+        </collision>
+    </link>
+    <joint name="motor_2_joint" type="fixed">
+        <origin xyz="${motor_placement_radius * cos_4_3_pi * in_m} ${motor_placement_radius * sin_4_3_pi *in_m} ${-motor_height/2 *in_m}" rpy="0 0 ${(4*pi)/3}" />
         <parent link="base_link"/>
-        <child link="right_wheel_link"/>
-        <axis xyz="0 1 0"/>
+        <child link="motor_2_link" />
+    </joint>
+    <!-- wheel 2 -->
+    <link name="wheel_2_link">
+        <inertial>
+            <origin xyz="0 0 0"/>
+            <mass value=".5" />
+            <inertia ixx="0.001" ixy="0.0" ixz="0.0"
+            iyy="0.001" iyz="0.0" izz="0.001" />
+        </inertial>
+        <visual>
+            <origin xyz="0 0 0" rpy="0 ${pi/2} 0" />
+            <geometry>
+                <cylinder radius="${wheel_radius*in_m}" length = "${wheel_width*in_m}"/>
+            </geometry>
+            <material name="Green" />
+        </visual>
+        <collision>
+            <origin xyz="0 0 0" rpy="0 ${pi/2} 0" />
+            <geometry>
+                <cylinder radius="${wheel_radius*in_m}" length = "${wheel_width*in_m}"/>
+            </geometry>
+        </collision>
+    </link>
+    <joint name="wheel_2_joint" type="continuous">
+        <origin xyz="${wheel_axil_offset * in_m} 0 0" rpy="0 0 0"/>
+        <parent link="motor_2_link"/>
+        <child link="wheel_2_link"/>
+        <axis xyz="1 0 0"/>
     </joint>
 </robot>
