Commit message: finished tentitive urdf

File: mesh_bot_description/urdf/mesh_bot.urdf.xacro (robot description, xacro)
@@ -1,3 +1,4 @@
 <?xml version="1.0"?>
+<!-- Writen by James Anderson 3/13/12-->
 <robot name="jomegatron"
     xmlns:sensor="http://playerstage.sourceforge.net/gazebo/xmlschema/#sensor"
@@ -11,40 +12,29 @@
     <property name="cos_4_3_pi" value="-0.5"/>
     <property name="sin_4_3_pi" value="-0.866025"/>
-    <property name="base_radius" value="12"/>
+    <property name="cos_1_3_pi" value="0.5"/>
+    <property name="sin_1_3_pi" value="0.866"/>
+    <property name="cos_pi" value="-1"/>
+    <property name="sin_pi" value="0"/>
+    <property name="cos_5_3_pi" value="0.5"/>
+    <property name="sin_5_3_pi" value="-0.866"/>
+    <property name="base_radius" value="10"/>
     <property name="base_height" value=".5"/>
-    <!-- motors are in inches -->
+    <property name="platform_1_height" value="5"/>
+    <property name="platform_2_height" value="19"/>
+    <property name="platform_3_height" value="23.5"/>
     <property name="motor_height" value="2"/>
     <property name="motor_width" value="2"/>
     <property name="motor_length" value="4"/>
-    <property name="motor_placement_radius" value="6"/>
-    <!-- wheels are in inches-->
+    <property name="motor_placement_radius" value="5"/>
     <property name="wheel_radius" value="2"/>
     <property name="wheel_width" value="1"/>
     <property name="wheel_axil_offset" value="1.5"/>
-    <property name="castor_bar_height" value="6"/>
-    <property name="castor_bar_width" value="4"/>
-    <property name="castor_bar_length" value="5"/>
-    <property name="castor_bar_setback" value="25"/>
-    <property name="castor_radius" value="3"/>
-    <property name="castor_width" value="3"/>
-    <property name="castor_radius" value="4"/>
-    <property name="mast_base_height" value="16"/>
-    <property name="mast_base_width" value="28"/>
-    <property name="mast_base_length" value="1"/>
-    <property name="mast_base_setback" value="13"/>
-    <property name="mast_vertical_height" value="5"/>
-    <property name="mast_vertical_width" value="1"/>
-    <property name="mast_vertical_length" value="1"/>
-    <property name="mast_horizontal_height" value="1"/>
-    <property name="mast_horizontal_width" value="1"/>
-    <property name="mast_horizontal_length" value="12"/>
-    <property name="mast_horizontal_setback" value="8"/>
-    <property name="camera_mount_height" value="3.5"/>
-    <property name="camera_mount_width" value="3.5"/>
-    <property name="camera_mount_length" value="1"/>
-    <property name="camera_mount_setback" value="1"/>
-    <property name="pt_grey_height" value="2"/>
-    <property name="pt_grey_width" value="3"/>
-    <property name="pt_grey_length" value="1.5"/>
+    <property name="rod_height" value="24"/>
+    <property name="rod_radius" value="0.25"/>
+    <property name="rod_placement_radius" value="9"/>
+    <property name="kinect_base_height" value="1"/>
+    <property name="kinect_joint_height" value="1"/>
+    <property name="kinect_joint_setback" value="1"/>
+    <property name="kinect_placement_radius" value="8"/>
     <material name="Green">
         <color rgba="0.0 0.8 0.0 1.0"/>
@@ -78,5 +68,5 @@
             <origin xyz="0 0 0" rpy="0 0 0" />
             <geometry>
-                <cylinder radius="${base_radius*in_m}" length = ".01"/>
+                <cylinder radius="${base_radius*in_m}" length = ".001"/>
             </geometry>
         </collision>
@@ -109,4 +99,173 @@
         <parent link="base_footprint"/>
         <child link="base_link" />
+    </joint>
+    <!-- platform 1 -->
+    <link name="platform_1_link">
+        <inertial>
+          <mass value="5" />
+          <origin xyz="0 0 0" />
+          <inertia ixx="0.0001" ixy="0.0" ixz="0.0"
+                  iyy="0.0001" iyz="0.0"
+                  izz="0.0001" />
+        </inertial>
+        <visual>
+            <origin xyz="0 0 ${(base_height/2)*in_m}" rpy="0 0 0" />
+            <geometry>
+                <cylinder radius="${base_radius*in_m}" length = "${base_height*in_m}"/>
+            </geometry>
+            <material name="Grey" />
+        </visual>
+        <collision>
+            <origin xyz="0 0 ${(base_height/2)*in_m}" rpy="0 0 0" />
+            <geometry>
+                <cylinder radius="${base_radius*in_m}" length = "${base_height*in_m}"/>
+            </geometry>
+        </collision>
+    </link>
+    <joint name="platform_1_joint" type="fixed">
+        <origin xyz="0 0 ${platform_1_height*in_m}" rpy="0 0 0" />
+        <parent link="base_link"/>
+        <child link="platform_1_link" />
+    </joint>
+    <!-- platform 2 -->
+    <link name="platform_2_link">
+        <inertial>
+          <mass value="5" />
+          <origin xyz="0 0 0" />
+          <inertia ixx="0.0001" ixy="0.0" ixz="0.0"
+                  iyy="0.0001" iyz="0.0"
+                  izz="0.0001" />
+        </inertial>
+        <visual>
+            <origin xyz="0 0 ${(base_height/2)*in_m}" rpy="0 0 0" />
+            <geometry>
+                <cylinder radius="${base_radius*in_m}" length = "${base_height*in_m}"/>
+            </geometry>
+            <material name="Grey" />
+        </visual>
+        <collision>
+            <origin xyz="0 0 ${(base_height/2)*in_m}" rpy="0 0 0" />
+            <geometry>
+                <cylinder radius="${base_radius*in_m}" length = "${base_height*in_m}"/>
+            </geometry>
+        </collision>
+    </link>
+    <joint name="platform_2_joint" type="fixed">
+        <origin xyz="0 0 ${platform_2_height*in_m}" rpy="0 0 0" />
+        <parent link="base_link"/>
+        <child link="platform_2_link" />
+    </joint>
+    <!-- kinect -->
+    <link name="kinect_link">
+        <inertial>
+            <mass value="0.01" />
+            <origin xyz="0 0 0" />
+            <inertia ixx="0.001" ixy="0.0" ixz="0.0"
+                     iyy="0.001" iyz="0.0"
+                     izz="0.001" />
+        </inertial>
+        <visual>
+            <origin xyz=" ${kinect_joint_setback * in_m} 0 ${kinect_joint_height * in_m} " rpy="0 0 0" />
+            <geometry>
+                <mesh filename="package://mesh_bot_description/meshes/kinect.dae"/>
+            </geometry>
+        </visual>
+        <collision>
+            <origin xyz="0 0.0 ${kinect_joint_height * in_m}" rpy="0 0 0" />
+            <geometry>
+                <box size="0.0730 .2760 0.0720"/>
+            </geometry>
+        </collision>
+    </link>
+    <joint name="base_kinect_joint" type="continuous">
+        <origin xyz="${(kinect_placement_radius) * in_m} 0 ${(kinect_base_height + base_height)* in_m}"
+                rpy="0 0 0" />
+        <parent link="platform_2_link" />
+        <child link="kinect_link" />
+        <axis xyz="0 1 0"/>
+    </joint>
+    <joint name="kinect_depth_joint" type="fixed">
+        <origin xyz="${kinect_joint_setback * in_m} 0.018 ${kinect_joint_height * in_m}" rpy="0 0 0" />
+        <parent link="kinect_link" />
+        <child link="kinect_depth_frame" />
+    </joint>
+    <link name="kinect_depth_frame">
+        <inertial>
+            <mass value="0.01" />
+            <origin xyz="0 0 0" />
+            <inertia ixx="0.001" ixy="0.0" ixz="0.0"
+                     iyy="0.001" iyz="0.0"
+                     izz="0.001" />
+        </inertial>
+    </link>
+    <joint name="kinect_depth_optical_joint" type="fixed">
+        <origin xyz="0 0 0" rpy="${-pi/2} 0 ${-pi/2}" />
+        <parent link="kinect_depth_frame" />
+        <child link="kinect_depth_optical_frame" />
+    </joint>
+    <link name="kinect_depth_optical_frame">
+        <inertial>
+            <mass value="0.001" />
+            <origin xyz="0 0 0" />
+            <inertia ixx="0.0001" ixy="0.0" ixz="0.0"
+                     iyy="0.0001" iyz="0.0"
+                     izz="0.0001" />
+        </inertial>
+    </link>
+    <joint name="kinect_rgb_joint" type="fixed">
+        <origin xyz="${kinect_joint_setback * in_m} -0.005 ${kinect_joint_height * in_m}" rpy="0 0 0" />
+        <parent link="kinect_link" />
+        <child link="kinect_rgb_frame" />
+    </joint>
+    <link name="kinect_rgb_frame">
+        <inertial>
+            <mass value="0.001" />
+            <origin xyz="0 0 0" />
+            <inertia ixx="0.0001" ixy="0.0" ixz="0.0"
+                     iyy="0.0001" iyz="0.0"
+                     izz="0.0001" />
+        </inertial>
+    </link>
+    <joint name="kinect_rgb_optical_joint" type="fixed">
+        <origin xyz="0 0 0" rpy="${-pi/2} 0 ${-pi/2}" />
+        <parent link="kinect_rgb_frame" />
+        <child link="kinect_rgb_optical_frame" />
+    </joint>
+    <link name="kinect_rgb_optical_frame">
+        <inertial>
+            <mass value="0.001" />
+            <origin xyz="0 0 0" />
+            <inertia ixx="0.0001" ixy="0.0" ixz="0.0"
+                     iyy="0.0001" iyz="0.0"
+                     izz="0.0001" />
+        </inertial>
+    </link>
+    <!-- platform 3 -->
+    <link name="platform_3_link">
+        <inertial>
+          <mass value="5" />
+          <origin xyz="0 0 0" />
+          <inertia ixx="0.0001" ixy="0.0" ixz="0.0"
+                  iyy="0.0001" iyz="0.0"
+                  izz="0.0001" />
+        </inertial>
+        <visual>
+            <origin xyz="0 0 ${(base_height/2)*in_m}" rpy="0 0 0" />
+            <geometry>
+                <cylinder radius="${base_radius*in_m}" length = "${base_height*in_m}"/>
+            </geometry>
+            <material name="Grey" />
+        </visual>
+        <collision>
+            <origin xyz="0 0 ${(base_height/2)*in_m}" rpy="0 0 0" />
+            <geometry>
+                <cylinder radius="${base_radius*in_m}" length = "${base_height*in_m}"/>
+            </geometry>
+        </collision>
+    </link>
+    <joint name="platform_3_joint" type="fixed">
+        <origin xyz="0 0 ${platform_3_height*in_m}" rpy="0 0 0" />
+        <parent link="base_link"/>
+        <child link="platform_3_link" />
     </joint>
     <!-- motor 0 -->
@@ -278,3 +437,87 @@
         <axis xyz="1 0 0"/>
     </joint>
+    <!-- rod 0 -->
+    <link name="rod_0_link">
+        <inertial>
+            <origin xyz="0 0 0"/>
+            <mass value=".5" />
+            <inertia ixx="0.001" ixy="0.0" ixz="0.0"
+            iyy="0.001" iyz="0.0" izz="0.001" />
+        </inertial>
+        <visual>
+            <origin xyz="0 0 ${rod_height/2 * in_m}" rpy="0 0 0" />
+            <geometry>
+                <cylinder radius="${rod_radius*in_m}" length = "${rod_height*in_m}"/>
+            </geometry>
+            <material name="Grey" />
+        </visual>
+        <collision>
+            <origin xyz="0 0 ${rod_height/2 * in_m}" rpy="0 0 0" />
+            <geometry>
+                <cylinder radius="${rod_radius*in_m}" length = "${rod_height*in_m}"/>
+            </geometry>
+        </collision>
+    </link>
+    <joint name="rod_0_joint" type="fixed">
+        <origin xyz="${rod_placement_radius * cos_1_3_pi * in_m} ${rod_placement_radius * sin_1_3_pi * in_m} 0" rpy="0 0 0"/>
+        <parent link="base_link"/>
+        <child link="rod_0_link"/>
+        <axis xyz="0 0 1"/>
+    </joint>
+    <!-- rod 1 -->
+    <link name="rod_1_link">
+        <inertial>
+            <origin xyz="0 0 0"/>
+            <mass value=".5" />
+            <inertia ixx="0.001" ixy="0.0" ixz="0.0"
+            iyy="0.001" iyz="0.0" izz="0.001" />
+        </inertial>
+        <visual>
+            <origin xyz="0 0 ${rod_height/2 * in_m}" rpy="0 0 0" />
+            <geometry>
+                <cylinder radius="${rod_radius*in_m}" length = "${rod_height*in_m}"/>
+            </geometry>
+            <material name="Grey" />
+        </visual>
+        <collision>
+            <origin xyz="0 0 ${rod_height/2 * in_m}" rpy="0 0 0" />
+            <geometry>
+                <cylinder radius="${rod_radius*in_m}" length = "${rod_height*in_m}"/>
+            </geometry>
+        </collision>
+    </link>
+    <joint name="rod_1_joint" type="fixed">
+        <origin xyz="${-rod_placement_radius * in_m} 0 0" rpy="0 0 0"/>
+        <parent link="base_link"/>
+        <child link="rod_1_link"/>
+        <axis xyz="0 0 1"/>
+    </joint>
+    <!-- rod 2 -->
+    <link name="rod_2_link">
+        <inertial>
+            <origin xyz="0 0 0"/>
+            <mass value=".5" />
+            <inertia ixx="0.001" ixy="0.0" ixz="0.0"
+            iyy="0.001" iyz="0.0" izz="0.001" />
+        </inertial>
+        <visual>
+            <origin xyz="0 0 ${rod_height/2 * in_m}" rpy="0 0 0" />
+            <geometry>
+                <cylinder radius="${rod_radius*in_m}" length = "${rod_height*in_m}"/>
+            </geometry>
+            <material name="Grey" />
+        </visual>
+        <collision>
+            <origin xyz="0 0 ${rod_height/2 * in_m}" rpy="0 0 0" />
+            <geometry>
+                <cylinder radius="${rod_radius*in_m}" length = "${rod_height*in_m}"/>
+            </geometry>
+        </collision>
+    </link>
+    <joint name="rod_2_joint" type="fixed">
+        <origin xyz="${rod_placement_radius * cos_5_3_pi * in_m} ${rod_placement_radius * sin_5_3_pi * in_m} 0" rpy="0 0 0"/>
+        <parent link="base_link"/>
+        <child link="rod_2_link"/>
+        <axis xyz="0 0 1"/>
+    </joint>
 </robot>

Commit message: changed some dimensions little broken

File: mesh_bot_description/urdf/mesh_bot.urdf.xacro (robot description, xacro)
@@ -23,8 +23,11 @@
     <property name="platform_2_height" value="19"/>
     <property name="platform_3_height" value="23.5"/>
-    <property name="motor_height" value="2"/>
-    <property name="motor_width" value="2"/>
-    <property name="motor_length" value="4"/>
+    <property name="motor_height" value="0.0564 "/>
+    <property name="motor_width" value="0.0564 "/>
+    <property name="motor_length" value="0.082 "/>
     <property name="motor_placement_radius" value="5"/>
+    <property name="laptop_height" value="13"/>
+    <property name="laptop_width" value="16"/>
+    <property name="laptop_length" value="12"/>
     <property name="wheel_radius" value="2"/>
     <property name="wheel_width" value="1"/>
@@ -128,4 +131,32 @@
         <child link="platform_1_link" />
     </joint>
+    <!-- laptop -->
+    <link name="laptop_link">
+        <inertial>
+          <mass value="2" />
+          <origin xyz="0 0 0" />
+          <inertia ixx="0.0001" ixy="0.0" ixz="0.0"
+                  iyy="0.0001" iyz="0.0"
+                  izz="0.0001" />
+        </inertial>
+        <visual>
+            <origin xyz="${(laptop_height/2) * in_m} 0 0" rpy="0 0 0" />
+            <geometry>
+                <box size="${laptop_length * in_m} ${laptop_width * in_m} ${laptop_height * in_m}" />
+            </geometry>
+            <material name="Black" />
+        </visual>
+        <collision>
+            <origin xyz="${(laptop_height/2) * in_m} 0 0" rpy="0 0 0" />
+            <geometry>
+                <box size="${laptop_length * in_m} ${laptop_width * in_m} ${laptop_height * in_m}" />
+            </geometry>
+        </collision>
+    </link>
+    <joint name="laptop_joint" type="fixed">
+        <origin xyz="0 0 ${base_height *in_m}" rpy="0 0 0" />
+        <parent link="platform_1_link"/>
+        <child link="laptop_link" />
+    </joint>
     <!-- platform 2 -->
     <link name="platform_2_link">
@@ -279,19 +310,19 @@
         </inertial>
         <visual>
-            <origin xyz="${-motor_length/2 * in_m} 0 0" rpy="0 0 0" />
-            <geometry>
-                <box size="${motor_length *in_m} ${motor_width*in_m} ${motor_height*in_m}" />
+            <origin xyz="${-motor_length/2 } 0 0" rpy="0 0 0" />
+            <geometry>
+                <box size="${motor_length } ${motor_width} ${motor_height}" />
             </geometry>
             <material name="Black" />
         </visual>
         <collision>
-            <origin xyz="${-motor_length/2 * in_m} 0 0" rpy="0 0 0" />
-            <geometry>
-                <box size="${motor_length *in_m} ${motor_width*in_m} ${motor_height*in_m}" />
+            <origin xyz="${-motor_length/2 } 0 0" rpy="0 0 0" />
+            <geometry>
+                <box size="${motor_length } ${motor_width} ${motor_height}" />
             </geometry>
         </collision>
     </link>
     <joint name="motor_0_joint" type="fixed">
-        <origin xyz="${motor_placement_radius * in_m} 0 ${-motor_height/2 *in_m}" rpy="0 0 0" />
+        <origin xyz="${motor_placement_radius * in_m} 0 ${-motor_height/2 }" rpy="0 0 0" />
         <parent link="base_link"/>
         <child link="motor_0_link" />
@@ -335,19 +366,19 @@
         </inertial>
         <visual>
-            <origin xyz="${-motor_length/2 * in_m} 0 0" rpy="0 0 0" />
-            <geometry>
-                <box size="${motor_length *in_m} ${motor_width*in_m} ${motor_height*in_m}" />
+            <origin xyz="${-motor_length/2 } 0 0" rpy="0 0 0" />
+            <geometry>
+                <box size="${motor_length } ${motor_width} ${motor_height}" />
             </geometry>
             <material name="Black" />
         </visual>
         <collision>
-            <origin xyz="${-motor_length/2 * in_m} 0 0" rpy="0 0 0" />
-            <geometry>
-                <box size="${motor_length *in_m} ${motor_width*in_m} ${motor_height*in_m}" />
+            <origin xyz="${-motor_length/2 } 0 0" rpy="0 0 0" />
+            <geometry>
+                <box size="${motor_length } ${motor_width} ${motor_height}" />
             </geometry>
         </collision>
     </link>
     <joint name="motor_1_joint" type="fixed">
-        <origin xyz="${motor_placement_radius * cos_2_3_pi * in_m} ${motor_placement_radius * sin_2_3_pi *in_m} ${-motor_height/2 *in_m}" rpy="0 0 ${(2*pi)/3}" />
+        <origin xyz="${motor_placement_radius * cos_2_3_pi * in_m} ${motor_placement_radius * sin_2_3_pi *in_m} ${-motor_height/2 }" rpy="0 0 ${(2*pi)/3}" />
         <parent link="base_link"/>
         <child link="motor_1_link" />
@@ -391,19 +422,19 @@
         </inertial>
         <visual>
-            <origin xyz="${-motor_length/2 * in_m} 0 0" rpy="0 0 0" />
-            <geometry>
-                <box size="${motor_length *in_m} ${motor_width*in_m} ${motor_height*in_m}" />
+            <origin xyz="${-motor_length/2 } 0 0" rpy="0 0 0" />
+            <geometry>
+                <box size="${motor_length } ${motor_width} ${motor_height}" />
             </geometry>
             <material name="Black" />
         </visual>
         <collision>
-            <origin xyz="${-motor_length/2 * in_m} 0 0" rpy="0 0 0" />
-            <geometry>
-                <box size="${motor_length *in_m} ${motor_width*in_m} ${motor_height*in_m}" />
+            <origin xyz="${-motor_length/2 } 0 0" rpy="0 0 0" />
+            <geometry>
+                <box size="${motor_length } ${motor_width} ${motor_height}" />
             </geometry>
         </collision>
     </link>
     <joint name="motor_2_joint" type="fixed">
-        <origin xyz="${motor_placement_radius * cos_4_3_pi * in_m} ${motor_placement_radius * sin_4_3_pi *in_m} ${-motor_height/2 *in_m}" rpy="0 0 ${(4*pi)/3}" />
+        <origin xyz="${motor_placement_radius * cos_4_3_pi * in_m} ${motor_placement_radius * sin_4_3_pi *in_m} ${-motor_height/2 }" rpy="0 0 ${(4*pi)/3}" />
         <parent link="base_link"/>
         <child link="motor_2_link" />

Commit message: fixed controll code

File: mesh_bot_description/urdf/mesh_bot.urdf.xacro (robot description, xacro)
@@ -132,5 +132,5 @@
     </joint>
     <!-- laptop -->
-    <link name="laptop_link">
+    <!--link1 name="laptop_link">
         <inertial>
           <mass value="2" />
@@ -158,5 +158,5 @@
         <parent link="platform_1_link"/>
         <child link="laptop_link" />
-    </joint>
+    </joint-->
     <!-- platform 2 -->
     <link name="platform_2_link">

Commit message: fixed odometry and controll directions

File: mesh_bot_description/urdf/mesh_bot.urdf.xacro (robot description, xacro)
@@ -18,9 +18,9 @@
     <property name="cos_5_3_pi" value="0.5"/>
     <property name="sin_5_3_pi" value="-0.866"/>
-    <property name="base_radius" value="10"/>
+    <property name="base_radius" value="13"/>
     <property name="base_height" value=".5"/>
-    <property name="platform_1_height" value="5"/>
-    <property name="platform_2_height" value="19"/>
-    <property name="platform_3_height" value="23.5"/>
+    <property name="platform_1_height" value="15"/>
+    <property name="platform_2_height" value="32"/>
+    <property name="platform_3_height" value="36"/>
     <property name="motor_height" value="0.0564 "/>
     <property name="motor_width" value="0.0564 "/>
@@ -32,6 +32,6 @@
     <property name="wheel_radius" value="2"/>
     <property name="wheel_width" value="1"/>
-    <property name="wheel_axil_offset" value="1.5"/>
-    <property name="rod_height" value="24"/>
+    <property name="wheel_axil_offset" value="2"/>
+    <property name="rod_height" value="36"/>
     <property name="rod_radius" value="0.25"/>
     <property name="rod_placement_radius" value="9"/>
@@ -39,5 +39,5 @@
     <property name="kinect_joint_height" value="1"/>
     <property name="kinect_joint_setback" value="1"/>
-    <property name="kinect_placement_radius" value="8"/>
+    <property name="kinect_placement_radius" value="4.5"/>
     <material name="Green">
         <color rgba="0.0 0.8 0.0 1.0"/>
@@ -99,5 +99,5 @@
     </link>
     <joint name="base_footprint_joint" type="fixed">
-        <origin xyz="0 0 ${(motor_height/2 + wheel_radius)*in_m}" rpy="0 0 0" />
+        <origin xyz="0 0 ${motor_height/2 + wheel_radius * in_m}" rpy="0 0 0" />
         <parent link="base_footprint"/>
         <child link="base_link" />
